File: EFM_VCF6c.brd (EAGLE design)
At the start: 100 x 80 mm, 69 parts, among them IC2 LM13700N, Q1 2N3904, Q2 2N3904, Q3 2N3906, Q4 2N3904, Q6 2N3904, U1 POWER

Commit message: layout close
Parts:
- removed FREQ_INIT: 100k, rcl:RTRIM64W
- removed IC2: LM13700N, synthdiy updated imperial:DIL16
- removed IN1, IN2: LSP10, solpad:LSP10
- removed Q6: 2N3904, transistor-npn:TO92
- removed R1: 470k, rcl:0207/7
- removed R13, R14: 220k, rcl:0207/7
- removed R2, R4: 10k, rcl:0207/7
- removed R21: 220, rcl:0207/7
- removed R3: 1k, rcl:0207/7
- removed R5: 100k, rcl:0207/7
- added CUTOFF_INIT: 100k, rcl:RTRIM64W
- added IC1: LM13700N, synthdiy updated imperial:DIL16
- added IN_1, IN_2: LSP10, solpad:LSP10
- added Q5: 2N3906, transistor-pnp:TO92
- added R24, R25: 220k, rcl:0207/7
- added R26: 47k, rcl:0207/7
- added R27: 1M, rcl:0207/7
- added R28, R29: 10k, rcl:0207/7
- added R30: 100k, rcl:0207/7
- added R31: 220, rcl:0207/7
- C10: value 0.1uF -> 220uF; device rcl:C025-030X050 -> rcl:B45181A
- C12: value 220uF -> 10uF
- C3, C4: value 10uF -> 0.1uF; device rcl:B45181A -> rcl:C025-030X050
- C5: value 0.1uF -> 10uF; device rcl:C025-030X050 -> rcl:B45181A
- Q3: value 2N3906 -> 2N3904; device transistor-pnp:TO92 -> transistor-npn:TO92
- R12, R18: value 10k -> 1k
- R15: value 1M -> 1k
- R16: value 1k -> 10k; device rcl:0207/7 -> rcl:0309/12
- R17: value 100k -> 1k
- R19: value 47k -> 1k
- R20: value 100k -> 10k
- R22: value 10k -> 470k
- R23: value 1k -> 10k
- R6, R7: value 1k -> 100k
- moved CV2 167.3 mm to (63.5, 7.62)
- moved D1 150.1 mm to (73.7, 66.0)
- moved CV1 149.6 mm to (47.0, 7.62)
- moved CV1_NORM 142.6 mm to (74.9, 35.6)
- moved Q3 137.3 mm to (57.8, 46.4)
- moved D9 136.5 mm to (58.4, 58.4)
- moved RES_CV 136.1 mm to (47.0, 16.5)
- moved R11 135.5 mm to (38.1, 19.1), turned to 90 degrees
- moved R19 134.9 mm to (34.3, 19.1), turned to 90 degrees
- moved C12 132.1 mm to (40.6, 43.2), turned to 180 degrees
- moved R8 131.8 mm to (58.4, 10.2), turned to 270 degrees
- moved R12 130.1 mm to (16.5, 11.4), turned to 180 degrees
- moved R16 127.8 mm to (71.1, 47.0), turned to 180 degrees
- moved R17 127.3 mm to (61.6, 50.2), turned to 270 degrees
- moved R6 126.8 mm to (72.4, 10.2), turned to 270 degrees
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Connections:
- net +12V: now also C1.+, C3.1, CUTOFF_INIT.3, D7.A, IC1.11, R16.1, R20.1, R27.1; no longer C3.+, C5.1, D2.A, FREQ_INIT.3, IC2.11, R12.1, R15.1, R4.1
- net -12V: now also C2.-, C4.2, CUTOFF_INIT.1, IC1.6, Q2.1, R23.2, R29.2; no longer C4.-, C6.2, FREQ_INIT.1, IC2.6, Q6.1, R18.2, R2.2
- net GND: now also C1.-, C10.-, C2.+, C3.2, C4.1, IC1.13, Q3.3, Q5.2, R22.2, R26.2, R31.2; no longer C12.-, C3.-, C4.+, C5.2, C6.1, IC2.13, Q2.3, Q3.2, R1.2, R16.2, R21.2
- net N$1: now also IC1.1, R22.1; no longer IC2.1, R1.1
- net N$10: now also R8.2; no longer R11.2
- net N$11: now also IC1.5, IC1.7, R30.1; no longer IC2.5, IC2.7, R20.1
- net N$12: now also C6.1, IC1.3; no longer C10.1, IC2.3
- net N$13: now also C7.1
- net N$14: now also D4.C, D5.A; no longer D5.C, D6.A
- net N$16: now also Q2.2, R12.1, R6.1, R7.1, R8.1; no longer Q6.2, R10.1, R17.1, R23.1, R9.1
- net N$17: now also C9.1; no longer C7.1
- net N$18: now also C9.2, D5.C, D6.A; no longer C7.2, D6.C, D7.A
- net N$19: now also D6.C; no longer D7.C
- net N$2: now also R25.2; no longer R14.2
- net N$21: now also D2.A; no longer D3.A
- net N$22: now also D7.C; no longer D2.C
- net N$23: now also R24.2; no longer R13.2
- net N$24: now also Q5.3, R24.1, R25.1, R27.2; no longer Q3.3, R13.1, R14.1, R15.2
- net N$25: now also C10.+, R15.2, R18.2, R19.1, R20.2; no longer C12.+, R12.2, R16.1, R6.2, R7.2
- net N$26: now also R18.1; no longer R7.1
- net N$27: now also CUTOFF_INIT.2, R11.2; no longer FREQ_INIT.2, R17.2
- net N$28: now also C12.+, IC1.8, R29.1; no longer C1.+, IC2.8, R2.1
- net N$29: now also C7.2, D3.C, D4.A; no longer C9.2, D4.C, D5.A
- net N$3: now also Q3.1, R17.2; no longer Q2.1, R3.2
- net N$30: now also IC1.14, R30.2, R31.1; no longer IC2.14, R20.2, R21.1
- net N$31: now also C12.-; no longer C1.-
- net N$32: now also IC1.16, R28.1; no longer IC2.16, R22.1
- net N$33: now also Q5.1, R28.2; no longer Q3.1, R22.2
- net N$34: now also IN_2.MP; no longer IN2.MP
- net N$35: now also IC1.9, R23.1; no longer IC2.9, R18.1
- net N$36: now also IC1.10, IC1.12, R26.1; no longer IC2.10, IC2.12, R19.1
- net N$37: now also R12.2; no longer R23.2
- net N$4: now also R17.1; no longer R3.1
- net N$5: now also R10.2; no longer R5.2
- net N$53: now also R7.2; no longer R10.2
- net N$56: now also R6.2; no longer R9.2
- net N$57: now also R9.1; no longer R8.1
- net N$58: now also IN_1.MP; no longer IN1.MP
- net N$6: now also C5.-, R10.1, R9.2; no longer C2.-, R5.1, R8.2
- net N$7: now also C5.+, R15.1; no longer C2.+, R6.1
- net N$8: now also Q2.3, Q3.2, R16.2; no longer Q2.2, Q6.3, R4.2
- net N$9: now also C6.2, D2.C, D3.A, IC1.4; no longer C10.2, D3.C, D4.A, IC2.4
