File: EFM_VCF6c.sch (EAGLE design)
At the start: 52 parts, among them IC1 TL072P, IC2 LM13700N, Q1 2N3904, Q2 2N3904, Q3 2N3906, Q4 2N3904, Q5 2N3906, Q6 2N3906, U1 POWER

Commit message: schemo progress
Parts:
- added C11: 10uF, rcl:CPOL-USB45181A
- added C12: 220uF, rcl:CPOL-USB45181A
- added R12: 10k, rcl:R-US_0207/7
- added R6, R7: 1k, rcl:R-US_0207/7
- C2: value 22uF -> 10uF
Connections:
- new net N$11: C9.2, D4.C, D5.A
- new net N$12: C10.1, D8.C, D9.A
- new net N$13: D10.A, D9.C
- new net N$14: C8.2, D5.C, D6.A
- new net N$15: C8.1, D10.C, D11.A
- new net N$17: C7.1, D11.C, D12.A
- new net N$18: C7.2, D6.C, D7.A
- new net N$19: D7.C, Q1.C
- new net N$20: D12.C, Q4.C
- new net N$21: D1.C, D3.A
- new net N$22: D2.C, D8.A
- new net N$9: C10.2, D3.C, D4.A
- net +12V: now also D1.A, D2.A, R12.1
- net N$16: now also Q6.B, R10.1, R11.1
Other:
- moved on the sheet: C2, IN1, IN1_LEVEL, IN2, IN2_LEVEL, R5, R8

Commit message: layout begins
Parts:
- removed 24DB_OUT: LSP10, solpad:LSP10
- removed FREQ_TRIM: 100k, rcl:R-TRIMM64W
- removed IC1: TL072P, linear:TL072P
- removed Q5: 2N3906, transistor-pnp:2N3906
- added FREQ_INIT: 100k, rcl:R-TRIMM64W
- added OUT, RES_CV: LSP10, solpad:LSP10
- added R13, R14: 220k, rcl:R-US_0207/7
- added R15: 1M, rcl:R-US_0207/7
- added R16, R23: 1k, rcl:R-US_0207/7
- added R17, R20: 100k, rcl:R-US_0207/7
- added R18, R22: 10k, rcl:R-US_0207/7
- added R19: 47k, rcl:R-US_0207/7
- added R21: 220, rcl:R-US_0207/7
- added RESONANCE: 100k, pot:3RP/1610N
- added SCALE_TRIM: 2k, rcl:R-TRIMM64W
- C1: value 22uF -> 10uF
- C3, C4: value 0.1uF -> 10uF; device rcl:C-US025-030X050 -> rcl:CPOL-USB45181A
- Q6: value 2N3906 -> 2N3904; device transistor-pnp:2N3906 -> transistor-npn:2N3904
- R9: value 150k -> 100k
Connections:
- new net N$11: IC2A.OUT, IC2G$3.IN, R20.1
- new net N$2: R14.2, RES_CV.MP
- new net N$23: R13.2, RESONANCE.S
- new net N$24: Q3.E, R13.1, R14.1, R15.2
- new net N$25: C12.+, R12.2, R16.1, R6.2, R7.2
- new net N$26: C11.+, Q4.B, R7.1
- new net N$27: FREQ_INIT.S, R17.2
- new net N$28: C1.+, IC2G$3.OUT, R2.1
- new net N$30: IC2B.+IN, R20.2, R21.1
- new net N$31: C1.-, OUT.MP
- new net N$32: IC2B.IABC, R22.1
- new net N$33: Q3.C, R22.2
- new net N$35: C11.-, IC2G$4.OUT, R18.1
- new net N$36: IC2B.OUT, IC2G$4.IN, R19.1
- new net N$37: R23.2, SCALE_TRIM.S
- net +12V: now also C3.+, FREQ_INIT.E, R15.1, RESONANCE.E; no longer C3.1, FREQ_TRIM.E, IC1P.V+
- net -12V: now also C4.-, FREQ_INIT.A, R18.2; no longer C4.2, FREQ_TRIM.A, IC1P.V-
- net GND: now also C12.-, C3.-, C4.+, IC2B.-IN, Q3.B, R16.2, R19.2, R21.2, RESONANCE.A, SCALE_TRIM.E; no longer C3.2, C4.1, Q3.E
- net N$12: now also IC2A.+IN
- net N$16: now also R17.1, R23.1
- net N$7: now also R6.1
- net N$9: now also IC2A.-IN
Other:
- moved on the sheet: C1, C12, C5, C6, CUTOFF, CV1, CV1_LEVEL, CV1_NORM, CV2, CV2_LEVEL, IC2B, IN1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

Commit message: layout close
Parts:
- removed Q6: 2N3904, transistor-npn:2N3904
- removed R1: 470k, rcl:R-US_0207/7
- removed R3: 1k, rcl:R-US_0207/7
- removed R4: 10k, rcl:R-US_0207/7
- removed R5: 100k, rcl:R-US_0207/7
- added Q5: 2N3906, transistor-pnp:2N3906
- added R26: 47k, rcl:R-US_0207/7
- added R27: 1M, rcl:R-US_0207/7
- added R28: 10k, rcl:R-US_0207/7
- added R30: 100k, rcl:R-US_0207/7
- C10: value 0.1uF -> 220uF; device rcl:C-US025-030X050 -> rcl:CPOL-USB45181A
- C12: value 220uF -> 10uF
- C3, C4: value 10uF -> 0.1uF; device rcl:CPOL-USB45181A -> rcl:C-US025-030X050
- C5: value 0.1uF -> 10uF; device rcl:C-US025-030X050 -> rcl:CPOL-USB45181A
- Q3: value 2N3906 -> 2N3904; device transistor-pnp:2N3906 -> transistor-npn:2N3904
- R12, R18: value 10k -> 1k
- R15: value 1M -> 1k
- R16: value 1k -> 10k; device rcl:R-US_0207/7 -> rcl:R-US_0309/12
- R17: value 100k -> 1k
- R19: value 47k -> 1k
- R20: value 100k -> 10k
- R22: value 10k -> 470k
- R23: value 1k -> 10k
- R6, R7: value 1k -> 100k
- renumbered FREQ_INIT to CUTOFF_INIT, IC2 to IC1, IN1 to IN_1, IN2 to IN_2, R13 to R24, R14 to R25, R2 to R29, R21 to R31
Connections:
- net +12V: now also C1.+, C3.1, D7.A, R16.1, R20.1, R27.1; no longer C3.+, C5.1, D2.A, R12.1, R15.1, R4.1
- net -12V: now also C2.-, C4.2, Q2.C, R23.2; no longer C4.-, C6.2, Q6.C, R18.2
- net GND: now also C1.-, C10.-, C2.+, C3.2, C4.1, Q3.E, Q5.B, R22.2, R26.2; no longer C12.-, C3.-, C4.+, C5.2, C6.1, Q2.E, Q3.B, R1.2, R16.2
- net N$1: now also R22.1; no longer R1.1
- net N$10: now also R8.2; no longer R11.2
- net N$11: now also R30.1; no longer R20.1
- net N$12: now also C6.1; no longer C10.1
- net N$13: now also C7.1
- net N$14: now also D4.C, D5.A; no longer D5.C, D6.A
- net N$16: now also Q2.B, R12.1, R6.1, R7.1, R8.1; no longer Q6.B, R10.1, R17.1, R23.1, R9.1
- net N$17: now also C9.1; no longer C7.1
- net N$18: now also C9.2, D5.C, D6.A; no longer C7.2, D6.C, D7.A
- net N$19: now also D6.C; no longer D7.C
- net N$21: now also D2.A; no longer D3.A
- net N$22: now also D7.C; no longer D2.C
- net N$24: now also Q5.E, R27.2; no longer Q3.E, R15.2
- net N$25: now also C10.+, R15.2, R18.2, R19.1, R20.2; no longer C12.+, R12.2, R16.1, R6.2, R7.2
- net N$26: now also R18.1; no longer R7.1
- net N$27: now also R11.2; no longer R17.2
- net N$28: now also C12.+; no longer C1.+
- net N$29: now also C7.2, D3.C, D4.A; no longer C9.2, D4.C, D5.A
- net N$3: now also Q3.C, R17.2; no longer Q2.C, R3.2
- net N$30: now also R30.2; no longer R20.2
- net N$31: now also C12.-; no longer C1.-
- net N$32: now also R28.1; no longer R22.1
- net N$33: now also Q5.C, R28.2; no longer Q3.C, R22.2
- net N$35: now also R23.1; no longer R18.1
- net N$36: now also R26.1; no longer R19.1
- net N$37: now also R12.2; no longer R23.2
- net N$4: now also R17.1; no longer R3.1
- net N$5: now also R10.2; no longer R5.2
- net N$53: now also R7.2; no longer R10.2
- net N$56: now also R6.2; no longer R9.2
- net N$57: now also R9.1; no longer R8.1
- net N$6: now also C5.-, R10.1, R9.2; no longer C2.-, R5.1, R8.2
- net N$7: now also C5.+, R15.1; no longer C2.+, R6.1
- net N$8: now also Q2.E, Q3.B, R16.2; no longer Q2.B, Q6.E, R4.2
- net N$9: now also C6.2, D2.C, D3.A; no longer C10.2, D3.C, D4.A
Other:
- moved on the sheet: C1, C12, C2, C6, C7, C9, D2, D3, D4, D5, D6, D7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

Commit message: ready to test cut
Parts:
- R16: device rcl:R-US_0309/12 -> rcl:R-US_0207/7
Connections:
- net +12V renamed N$38
Changed lines of the file:
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@@
 <part name="R17" library="rcl" deviceset="R-US_" device="0207/7" value="1k"/>
 <part name="GND10" library="supply1" deviceset="GND" device=""/>
-<part name="R16" library="rcl" deviceset="R-US_" device="0309/12" value="10k"/>
+<part name="R16" library="rcl" deviceset="R-US_" device="0207/7" value="10k"/>
 <part name="P+7" library="supply1" deviceset="+12V" device=""/>
 <part name="P-5" library="supply1" deviceset="-12V" device=""/>
@@
 </segment>
 </net>
-<net name="+12V" class="0">
+<net name="N$38" class="0">
 <segment>
 <pinref part="U1" gate="G$1" pin="+12V"/>

Commit message: fix and mod for self res
Parts:
- Q3: value 2N3904 -> 2N3906; device transistor-npn:2N3904 -> transistor-pnp:2N3906
- R26: value 47k -> 100k
Connections:
- net -12V: now also Q3.C; no longer Q2.C
- net GND: now also Q4.E; no longer Q3.E
- net N$16: now also Q3.B; no longer Q2.B
- net N$20: now also Q2.C; no longer Q4.C
- net N$26: now also Q2.B; no longer Q4.B
- net N$3: now also Q4.C; no longer Q3.C
- net N$4: now also Q2.E; no longer Q4.E
- net N$8: now also Q3.E, Q4.B; no longer Q2.E, Q3.B
Other:
- moved on the sheet: C11, Q2, Q4, R16, R17
