File: EFM_VCF6c.sch (EAGLE design)
At the start: 74 parts, among them IC1 LM13700N, Q1 2N3904, Q2 2N3904, Q3 2N3906, Q4 2N3904, Q5 2N3906, U2 POWER

Commit message: routed and labels adjusted
Parts:
- removed C1, C2: 10uF, rcl:CPOL-USB45181A
- removed CV1_LEVEL, CV2_LEVEL, IN1_LEVEL, IN2_LEVEL: 100k, pot:3RP/1610N
- removed CV_IN2: AUDIO-JACKITEAD, erthenvar:AUDIO-JACKITEAD
- added CV1_LEV, CV2_LEV, IN1_LEV, IN2_LEV: 100k, bourns_ptd:PTD901
- added OUT: AUDIO-JACKITEAD, erthenvar:AUDIO-JACKITEAD
- C3, C4, C6, C7, C8, C9: value 0.1uF -> 100n
- CUTOFF, RESONANCE: device pot:3RP/1610N -> bourns_ptd:PTD901
- renumbered CV_IN1 to IN1
Connections:
- net -12V: no longer C2.-
- net GND: now also CV1_LEV.A, CV2_LEV.A, IN1_LEV.A, IN2_LEV.A, OUT.RING; no longer C1.-, C2.+, CV1_LEVEL.A, CV2_LEVEL.A, CV_IN2.RING, IN1_LEVEL.A, IN2_LEVEL.A
- net N$10: now also CV2_LEV.S; no longer CV2_LEVEL.S
- net N$31: now also OUT.TIP; no longer CV_IN2.TIP
- net N$34: now also IN2_LEV.E; no longer IN2_LEVEL.E
- net N$38: no longer C1.+
- net N$5: now also IN2_LEV.S; no longer IN2_LEVEL.S
- net N$53: now also CV1_LEV.S; no longer CV1_LEVEL.S
- net N$54: now also CV2_LEV.E; no longer CV2_LEVEL.E
- net N$57: now also IN1_LEV.S; no longer IN1_LEVEL.S
- net N$58: now also IN1_LEV.E; no longer IN1_LEVEL.E
- net N$59: now also CV1_LEV.E; no longer CV1_LEVEL.E
Other:
- moved on the sheet: C12, C22, C23, C24, C25, C3, C4, C6, C7, C8, C9, D13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
